Commit message: did stuff
Signed-off-by: FIRST_NAME LAST_NAME <MY_NAME@example.com>

File: linorobot2_description/urdf/mecanum_properties.urdf.xacro (robot description, xacro)
@@ -1,20 +1,20 @@
 <?xml version="1.0"?>
 <robot xmlns:xacro="http://ros.org/wiki/xacro">
-  <xacro:property name="base_length" value="0.445" />
-  <xacro:property name="base_width" value="0.200" />
-  <xacro:property name="base_height" value="0.129" />
-  <xacro:property name="base_mass" value="10" />
-  <xacro:property name="wheel_radius" value="0.07162" />
-  <xacro:property name="wheel_width" value="0.05" />
-  <xacro:property name="wheel_pos_x" value="0.120" />
-  <xacro:property name="wheel_pos_y" value="0.1355" />
-  <xacro:property name="wheel_pos_z" value="-0.04788" />
-  <xacro:property name="wheel_mass" value=".6" />
-  <xacro:property name="wheel_torque" value="20" />
+  <xacro:property name="base_length" value="0.16" />
+  <xacro:property name="base_width" value="0.156" />
+  <xacro:property name="base_height" value="0.01" />
+  <xacro:property name="base_mass" value="0.7" />
+  <xacro:property name="wheel_radius" value="0.043" />
+  <xacro:property name="wheel_width" value="0.0255" />
+  <xacro:property name="wheel_pos_x" value="-0.085" />
+  <xacro:property name="wheel_pos_y" value="0.11" />
+  <xacro:property name="wheel_pos_z" value="0.0345" />
+  <xacro:property name="wheel_mass" value="0.05" />
+  <xacro:property name="wheel_torque" value="0.088" />
   <xacro:property name="laser_pose">
-    <origin xyz="-0.0475 0 0.125" rpy="0 0 0"/>
+    <origin xyz="0.065 0 0.1960" rpy="0 0 0"/>
   </xacro:property>
   <xacro:property name="depth_sensor_pose">
-    <origin xyz="0.2375 0 0.06" rpy="0 0 0"/>
+    <origin xyz="0.057 0 0.1695" rpy="0 0 0"/>
   </xacro:property>
 </robot>

Commit message: Lol
Signed-off-by: FIRST_NAME LAST_NAME <MY_NAME@example.com>

File: linorobot2_description/urdf/mecanum_properties.urdf.xacro (robot description, xacro)
@@ -13,8 +13,8 @@
   <xacro:property name="wheel_torque" value="0.088" />
   <xacro:property name="laser_pose">
-    <origin xyz="0.065 0 0.1960" rpy="0 0 0"/>
+    <origin xyz="0.065 0 0.0" rpy="0 0 0"/>
   </xacro:property>
   <xacro:property name="depth_sensor_pose">
-    <origin xyz="0.057 0 0.1695" rpy="0 0 0"/>
+    <origin xyz="0.1695 0 0.05" rpy="0 0 0"/>
   </xacro:property>
 </robot>

Commit message: changes to new platform
Signed-off-by: git is a cats name <mrnic3@gmail.com>

File: linorobot2_description/urdf/mecanum_properties.urdf.xacro (robot description, xacro)
@@ -1,20 +1,20 @@
 <?xml version="1.0"?>
 <robot xmlns:xacro="http://ros.org/wiki/xacro">
-  <xacro:property name="base_length" value="0.16" />
-  <xacro:property name="base_width" value="0.156" />
-  <xacro:property name="base_height" value="0.01" />
+  <xacro:property name="base_length" value="0.155" />
+  <xacro:property name="base_width" value="0.183" />
+  <xacro:property name="base_height" value="0.045" />
   <xacro:property name="base_mass" value="0.7" />
-  <xacro:property name="wheel_radius" value="0.043" />
-  <xacro:property name="wheel_width" value="0.0255" />
+  <xacro:property name="wheel_radius" value="0.039" />
+  <xacro:property name="wheel_width" value="0.036" />
   <xacro:property name="wheel_pos_x" value="-0.085" />
   <xacro:property name="wheel_pos_y" value="0.11" />
-  <xacro:property name="wheel_pos_z" value="0.0345" />
+  <xacro:property name="wheel_pos_z" value="0.0" />
   <xacro:property name="wheel_mass" value="0.05" />
   <xacro:property name="wheel_torque" value="0.088" />
   <xacro:property name="laser_pose">
-    <origin xyz="0.065 0 0.0" rpy="0 0 0"/>
+    <origin xyz="0.0 0 0.085" rpy="0 0 0"/>
   </xacro:property>
   <xacro:property name="depth_sensor_pose">
-    <origin xyz="0.1695 0 0.05" rpy="0 0 0"/>
+    <origin xyz="0.075 0 0.05" rpy="0 0 0"/>
   </xacro:property>
 </robot>

Commit message: changed orientation of laser
Signed-off-by: git is a cats name <mrnic3@gmail.com>

File: linorobot2_description/urdf/mecanum_properties.urdf.xacro (robot description, xacro)
@@ -13,5 +13,5 @@
   <xacro:property name="wheel_torque" value="0.088" />
   <xacro:property name="laser_pose">
-    <origin xyz="0.0 0 0.085" rpy="0 0 0"/>
+    <origin xyz="0.0 0 0.085" rpy="0 0 1.5708"/>
   </xacro:property>
   <xacro:property name="depth_sensor_pose">

Commit message: tweaked settings
Signed-off-by: git is a cats name <mrnic3@gmail.com>

File: linorobot2_description/urdf/mecanum_properties.urdf.xacro (robot description, xacro)
@@ -2,11 +2,11 @@
 <robot xmlns:xacro="http://ros.org/wiki/xacro">
   <xacro:property name="base_length" value="0.155" />
-  <xacro:property name="base_width" value="0.183" />
+  <xacro:property name="base_width" value="0.164" />
   <xacro:property name="base_height" value="0.045" />
   <xacro:property name="base_mass" value="0.7" />
-  <xacro:property name="wheel_radius" value="0.039" />
-  <xacro:property name="wheel_width" value="0.036" />
-  <xacro:property name="wheel_pos_x" value="-0.085" />
-  <xacro:property name="wheel_pos_y" value="0.11" />
+  <xacro:property name="wheel_radius" value="0.024" />
+  <xacro:property name="wheel_width" value="0.025" />
+  <xacro:property name="wheel_pos_x" value="-0.082" />
+  <xacro:property name="wheel_pos_y" value="0.0651" />
   <xacro:property name="wheel_pos_z" value="0.0" />
   <xacro:property name="wheel_mass" value="0.05" />
